Commit message: some corrections

File: urdf/PAROL6.urdf (robot description, URDF)
Before this commit: robot PAROL6, 8 links, 7 joints
Joints:
- joint J1: origin xyz=0 0 0 rpy=0 0 0 -> xyz=0 0 0 rpy=0 0 -0.436
- joint J2: origin xyz=0.0234207210610375 0 0.1105 rpy=-1.5707963267949 0 0 -> xyz=0.0234207210610375 0 0.1105 rpy=-1.5707963267949 0.2 0
- joint J3: origin xyz=0 -0.18 0 rpy=3.1416 0 -1.5708 -> xyz=0 -0.18 0 rpy=3.1416 0 -3.1
- joint J5: origin xyz=0 0 0.17635 rpy=1.5708 0 0 -> xyz=0 0 0.17635 rpy=1.5708 0 0.045
- joint J6: origin xyz=0 0 0 rpy=-1.5708 0 0 -> xyz=0 0.039 0 rpy=-1.5708 0 0

File: urdf/gazebo.xacro (robot description, xacro)
@@ -71,11 +71,4 @@
       <state_interface name="effort"/>
     </joint>
-    <transmission name="transmission1">
-      <plugin>transmission_interface/SimpleTransmission</plugin>
-      <actuator name="actuator1" role="actuator1"/>
-      <joint name="J1" role="J1">
-        <mechanical_reduction>6.4</mechanical_reduction>
-      </joint>
-    </transmission>
   </ros2_control>
   <gazebo>
@@ -90,4 +83,5 @@
       <joint_name>J6</joint_name>
     </plugin>
+    <!--
     <plugin filename="libgz_ros2_control-system.so" name="gz_ros2_control::GazeboSimROS2ControlPlugin">
       <robot_param>robot_description</robot_param>
@@ -95,14 +89,67 @@
       <parameters>$(find parol6)/config/controller.yaml</parameters>
     </plugin>
-    <!-- Gazebo plugin can be used to control the joint directly.
+    -->
+    <!-- Gazebo plugin can be used to control the joint directly. -->
       <plugin
         filename="gz-sim-joint-position-controller-system"
         name="gz::sim::systems::JointPositionController">
         <joint_name>J1</joint_name>
-        <topic>J6</topic>
-        <p_gain>10</p_gain>
+        <topic>J1</topic>
+        <p_gain>5</p_gain>
         <i_gain>1</i_gain>
         <d_gain>0.1</d_gain>
+        <initial_position>0</initial_position>
       </plugin>
+      <plugin
+        filename="gz-sim-joint-position-controller-system"
+        name="gz::sim::systems::JointPositionController">
+        <joint_name>J2</joint_name>
+        <topic>J2</topic>
+        <p_gain>5</p_gain>
+        <i_gain>1</i_gain>
+        <d_gain>0.1</d_gain>
+        <initial_position>0</initial_position>
+      </plugin>
+      <plugin
+        filename="gz-sim-joint-position-controller-system"
+        name="gz::sim::systems::JointPositionController">
+        <joint_name>J3</joint_name>
+        <topic>J3</topic>
+        <p_gain>5</p_gain>
+        <i_gain>1</i_gain>
+        <d_gain>0.1</d_gain>
+        <initial_position>0</initial_position>
+      </plugin>
+      <plugin
+        filename="gz-sim-joint-position-controller-system"
+        name="gz::sim::systems::JointPositionController">
+        <joint_name>J4</joint_name>
+        <topic>J4</topic>
+        <p_gain>5</p_gain>
+        <i_gain>1</i_gain>
+        <d_gain>0.1</d_gain>
+        <initial_position>0</initial_position>
+      </plugin>
+      <plugin
+        filename="gz-sim-joint-position-controller-system"
+        name="gz::sim::systems::JointPositionController">
+        <joint_name>J5</joint_name>
+        <topic>J5</topic>
+        <p_gain>5</p_gain>
+        <i_gain>1</i_gain>
+        <d_gain>0.1</d_gain>
+        <initial_position>0</initial_position>
+      </plugin>
+      <plugin
+        filename="gz-sim-joint-position-controller-system"
+        name="gz::sim::systems::JointPositionController">
+        <joint_name>J6</joint_name>
+        <topic>J6</topic>
+        <p_gain>5</p_gain>
+        <i_gain>1</i_gain>
+        <d_gain>0.1</d_gain>
+        <initial_position>0</initial_position>
+      </plugin>
+    <!--
       However, it will overrides the control from ros2 side.
      -->
